Commit message: added hello_moveit = C++ move_group_interface example

File: src/doosan-robot2/dsr_description2/urdf/m1013.urdf (robot description, URDF)
Before this commit: robot m1013, 11 links, 10 joints
Links:
- removed link gripper
- removed link left_finger
- removed link right_finger
- added link world
Joints:
- removed joint gripper_joint
- removed joint left_finger_joint
- removed joint right_finger_joint
- added joint world_to_base_link: type fixed, parent world, child base_link, origin xyz=0 0 0 rpy=0 0 0
- joint joint_1: origin xyz=0 0 0.1525 rpy=0 0 3.14159 -> xyz=0 0 0.1525 rpy=0 0 0

File: src/doosan-robot2/dsr_moveit2/dsr_moveit_config_m1013/config/dsr.ros2_control.xacro (robot description, xacro)
@@ -61,22 +61,4 @@
                 </state_interface>
             </joint>
-            <joint name="left_finger_joint">
-                <command_interface name="position"/>
-                <state_interface name="position">
-                  <!-- <param name="initial_value">${initial_positions['left_finger_joint']}</param> -->
-                </state_interface>
-                <state_interface name="velocity">
-                    <param name="initial_value">0.0</param>
-                </state_interface>
-            </joint>
-            <joint name="right_finger_joint">
-                <command_interface name="position"/>
-                <state_interface name="position">
-                  <!-- <param name="initial_value">${initial_positions['right_finger_joint']}</param> -->
-                </state_interface>
-                <state_interface name="velocity">
-                    <param name="initial_value">0.0</param>
-                </state_interface>
-            </joint>
         </ros2_control>
     </xacro:macro>

Commit message: added joint_state merger, automatically select gripper depending on mode, added collision objects

File: src/doosan-robot2/dsr_description2/urdf/m1013.urdf (robot description, URDF)
Before this commit: robot m1013, 9 links, 8 joints
Links:
- added link gripper, mass 2.9; collision mesh filename=package://dsr_description2/meshes/m1013_gripper/gripper_col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 scale=1 1 1; visual mesh filename=package://dsr_description2/meshes/m1013_gripper/gripper_wo_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 scale=1 1 1
- added link left_finger, mass 0.1; collision mesh filename=package://dsr_description2/meshes/m1013_gripper/finger_left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 scale=1 1 1; visual mesh filename=package://dsr_description2/meshes/m1013_gripper/finger_left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 scale=1 1 1
- added link right_finger, mass 0.1; collision mesh filename=package://dsr_description2/meshes/m1013_gripper/finger_righ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 scale=1 1 1; visual mesh filename=package://dsr_description2/meshes/m1013_gripper/finger_righ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 scale=1 1 1
Joints:
- added joint gripper_joint: type fixed, parent link_6, child gripper, origin xyz=0 0 0 rpy=-1.571 3.14159 -1.571
- added joint left_finger_joint: type prismatic, parent gripper, child left_finger, axis 0 0 1, limit lower=0.0 upper=0.06 effort=100.0 velocity=0.2
- added joint right_finger_joint: type prismatic, parent gripper, child right_finger, origin xyz=0 0 0 rpy=0 0 0, axis 0 0 -1, limit lower=0.0 upper=0.06 effort=100.0 velocity=0.2, mimic joint=left_finger_joint multiplier=1.0 offset=0.0

File: src/doosan-robot2/dsr_moveit2/dsr_moveit_config_m1013/config/dsr.ros2_control.xacro (robot description, xacro)
@@ -61,4 +61,22 @@
                 </state_interface>
             </joint>
+                        <joint name="left_finger_joint">
+                <command_interface name="position"/>
+                <state_interface name="position">
+                  <!-- <param name="initial_value">${initial_positions['left_finger_joint']}</param> -->
+                </state_interface>
+                <state_interface name="velocity">
+                    <param name="initial_value">0.0</param>
+                </state_interface>
+            </joint>
+            <joint name="right_finger_joint">
+                <command_interface name="position"/>
+                <state_interface name="position">
+                  <!-- <param name="initial_value">${initial_positions['right_finger_joint']}</param> -->
+                </state_interface>
+                <state_interface name="velocity">
+                    <param name="initial_value">0.0</param>
+                </state_interface>
+            </joint>
         </ros2_control>
     </xacro:macro>
